Commit message: Added example file and logging

File: install/johnny_5_description/share/johnny_5_description/urdf/johnny_5.xacro (robot description, xacro)
@@ -1,232 +1 @@
-<?xml version="1.0"?>
-<!-- filepath: /home/matt/johnny_ws/src/johnny_5_description/urdf/johnny_5.xacro -->
-<robot name="johnny_5" xmlns:xacro="http://www.ros.org/wiki/xacro">
-  <!-- Define some constants for Johnny 5's proportions -->
-  <xacro:property name="base_width" value="0.35"/>
-  <xacro:property name="base_length" value="0.45"/>
-  <xacro:property name="base_height" value="0.12"/>
-  <!-- Track dimensions -->
-  <xacro:property name="track_width" value="0.08"/>
-  <xacro:property name="track_length" value="0.40"/>
-  <xacro:property name="track_height" value="0.15"/>
-  <xacro:property name="track_separation" value="0.30"/>
-  <!-- Upper body dimensions -->
-  <xacro:property name="torso_width" value="0.25"/>
-  <xacro:property name="torso_length" value="0.20"/>
-  <xacro:property name="torso_height" value="0.30"/>
-  <!-- Head dimensions -->
-  <xacro:property name="head_radius" value="0.12"/>
-  <!-- Arm dimensions -->
-  <xacro:property name="arm_length" value="0.25"/>
-  <xacro:property name="arm_radius" value="0.03"/>
-  <!-- Define inertial property macros -->
-  <xacro:macro name="box_inertia" params="m w h d">
-    <inertial>
-      <origin xyz="0 0 0" rpy="0 0 0"/>
-      <mass value="${m}"/>
-      <inertia ixx="${(m/12) * (h*h + d*d)}" ixy="0.0" ixz="0.0"
-               iyy="${(m/12) * (w*w + d*d)}" iyz="0.0"
-               izz="${(m/12) * (w*w + h*h)}"/>
-    </inertial>
-  </xacro:macro>
-  <xacro:macro name="cylinder_inertia" params="m r h">
-    <inertial>
-      <origin xyz="0 0 0" rpy="0 0 0" />
-      <mass value="${m}"/>
-      <inertia ixx="${(m/12) * (3*r*r + h*h)}" ixy="0" ixz="0"
-               iyy="${(m/12) * (3*r*r + h*h)}" iyz="0"
-               izz="${(m/2) * (r*r)}"/>
-    </inertial>
-  </xacro:macro>
-  <xacro:macro name="sphere_inertia" params="m r">
-    <inertial>
-      <mass value="${m}"/>
-      <inertia ixx="${(2/5) * m * (r*r)}" ixy="0.0" ixz="0.0"
-               iyy="${(2/5) * m * (r*r)}" iyz="0.0"
-               izz="${(2/5) * m * (r*r)}"/>
-    </inertial>
-  </xacro:macro>
-  <!-- Materials -->
-  <material name="silver">
-    <color rgba="0.7 0.7 0.7 1.0"/>
-  </material>
-  <material name="black">
-    <color rgba="0.1 0.1 0.1 1.0"/>
-  </material>
-  <material name="blue">
-    <color rgba="0.2 0.2 0.8 1.0"/>
-  </material>
-  <material name="red">
-    <color rgba="0.8 0.2 0.2 1.0"/>
-  </material>
-  <!-- Robot base/chassis -->
-  <link name="base_link">
-    <visual>
-      <geometry>
-        <box size="${base_length} ${base_width} ${base_height}"/>
-      </geometry>
-      <material name="silver"/>
-    </visual>
-    <collision>
-      <geometry>
-        <box size="${base_length} ${base_width} ${base_height}"/>
-      </geometry>
-    </collision>
-    <xacro:box_inertia m="20" w="${base_width}" d="${base_length}" h="${base_height}"/>
-  </link>
-  <!-- Robot Footprint -->
-  <link name="base_footprint"/>
-  <joint name="base_joint" type="fixed">
-    <parent link="base_link"/>
-    <child link="base_footprint"/>
-    <origin xyz="0.0 0.0 ${-track_height/2}" rpy="0 0 0"/>
-  </joint>
-  <!-- Track macro -->
-  <xacro:macro name="track" params="prefix y_reflect">
-    <link name="${prefix}_track">
-      <visual>
-        <origin xyz="0 0 0" rpy="0 0 0"/>
-        <geometry>
-          <box size="${track_length} ${track_width} ${track_height}"/>
-        </geometry>
-        <material name="black"/>
-      </visual>
-      <collision>
-        <origin xyz="0 0 0" rpy="0 0 0"/>
-        <geometry>
-          <box size="${track_length} ${track_width} ${track_height}"/>
-        </geometry>
-      </collision>
-      <xacro:box_inertia m="5" w="${track_width}" d="${track_length}" h="${track_height}"/>
-    </link>
-    <joint name="${prefix}_track_joint" type="continuous">
-      <parent link="base_link"/>
-      <child link="${prefix}_track"/>
-      <origin xyz="0 ${y_reflect*track_separation/2} ${-base_height/2-track_height/2}" rpy="0 0 0"/>
-      <axis xyz="1 0 0"/>  <!-- Tracks move forward/backward -->
-    </joint>
-  </xacro:macro>
-  <!-- Left and right tracks -->
-  <xacro:track prefix="left" y_reflect="1" />
-  <xacro:track prefix="right" y_reflect="-1" />
-  <!-- Upper torso -->
-  <link name="torso">
-    <visual>
-      <geometry>
-        <box size="${torso_length} ${torso_width} ${torso_height}"/>
-      </geometry>
-      <material name="silver"/>
-    </visual>
-    <collision>
-      <geometry>
-        <box size="${torso_length} ${torso_width} ${torso_height}"/>
-      </geometry>
-    </collision>
-    <xacro:box_inertia m="8" w="${torso_width}" d="${torso_length}" h="${torso_height}"/>
-  </link>
-  <joint name="torso_joint" type="revolute">
-    <parent link="base_link"/>
-    <child link="torso"/>
-    <origin xyz="0 0 ${base_height/2 + torso_height/2}" rpy="0 0 0"/>
-    <axis xyz="0 0 1"/>  <!-- Can rotate left/right -->
-    <limit lower="${-pi}" upper="${pi}" effort="10" velocity="1"/>
-  </joint>
-  <!-- Head -->
-  <link name="head">
-    <visual>
-      <geometry>
-        <sphere radius="${head_radius}"/>
-      </geometry>
-      <material name="silver"/>
-    </visual>
-    <collision>
-      <geometry>
-        <sphere radius="${head_radius}"/>
-      </geometry>
-    </collision>
-    <xacro:sphere_inertia m="2" r="${head_radius}"/>
-  </link>
-  <joint name="head_joint" type="revolute">
-    <parent link="torso"/>
-    <child link="head"/>
-    <origin xyz="0 0 ${torso_height/2 + head_radius}" rpy="0 0 0"/>
-    <axis xyz="0 0 1"/>  <!-- Head can turn -->
-    <limit lower="${-pi}" upper="${pi}" effort="5" velocity="2"/>
-  </joint>
-  <!-- Eyes (cameras) -->
-  <xacro:macro name="eye" params="prefix y_offset">
-    <link name="${prefix}_eye">
-      <visual>
-        <geometry>
-          <cylinder radius="0.02" length="0.03"/>
-        </geometry>
-        <material name="blue"/>
-      </visual>
-      <collision>
-        <geometry>
-          <cylinder radius="0.02" length="0.03"/>
-        </geometry>
-      </collision>
-      <xacro:cylinder_inertia m="0.1" r="0.02" h="0.03"/>
-    </link>
-    <joint name="${prefix}_eye_joint" type="revolute">
-      <parent link="head"/>
-      <child link="${prefix}_eye"/>
-      <origin xyz="${head_radius-0.01} ${y_offset} 0.02" rpy="0 ${pi/2} 0"/>
-      <axis xyz="0 0 1"/>
-      <limit lower="${-pi/4}" upper="${pi/4}" effort="1" velocity="1"/>
-    </joint>
-  </xacro:macro>
-  <xacro:eye prefix="left" y_offset="0.04" />
-  <xacro:eye prefix="right" y_offset="-0.04" />
-  <!-- Arms -->
-  <xacro:macro name="arm" params="prefix y_reflect">
-    <link name="${prefix}_arm">
-      <visual>
-        <origin xyz="${arm_length/2} 0 0" rpy="0 0 0"/>
-        <geometry>
-          <box size="${arm_length} ${arm_radius*2} ${arm_radius*2}"/>
-        </geometry>
-        <material name="silver"/>
-      </visual>
-      <collision>
-        <origin xyz="${arm_length/2} 0 0" rpy="0 0 0"/>
-        <geometry>
-          <box size="${arm_length} ${arm_radius*2} ${arm_radius*2}"/>
-        </geometry>
-      </collision>
-      <xacro:box_inertia m="1" w="${arm_radius*2}" d="${arm_length}" h="${arm_radius*2}"/>
-    </link>
-    <joint name="${prefix}_arm_joint" type="revolute">
-      <parent link="torso"/>
-      <child link="${prefix}_arm"/>
-      <origin xyz="0 ${y_reflect*(torso_width/2 + arm_radius)} ${torso_height/4}" rpy="0 0 0"/>
-      <axis xyz="0 1 0"/>  <!-- Arms can move up/down -->
-      <limit lower="${-pi/2}" upper="${pi/2}" effort="10" velocity="1"/>
-    </joint>
-    <!-- Hand/gripper -->
-    <link name="${prefix}_hand">
-      <visual>
-        <geometry>
-          <sphere radius="0.04"/>
-        </geometry>
-        <material name="red"/>
-      </visual>
-      <collision>
-        <geometry>
-          <sphere radius="0.04"/>
-        </geometry>
-      </collision>
-      <xacro:sphere_inertia m="0.2" r="0.04"/>
-    </link>
-    <joint name="${prefix}_hand_joint" type="revolute">
-      <parent link="${prefix}_arm"/>
-      <child link="${prefix}_hand"/>
-      <origin xyz="${arm_length} 0 0" rpy="0 0 0"/>
-      <axis xyz="1 0 0"/>
-      <limit lower="${-pi}" upper="${pi}" effort="2" velocity="2"/>
-    </joint>
-  </xacro:macro>
-  <xacro:arm prefix="left" y_reflect="1" />
-  <xacro:arm prefix="right" y_reflect="-1" />
-</robot>
+/home/matt/johnny_ws/src/johnny_5_description/urdf/johnny_5.xacro
